File: pcb_design/drivers.kicad_sch (KiCad schematic)
At the start: 21 parts, among them Q3 MMBT3906LT1G, U10 MCP2562-E-SN, U7 SN74LVC1G125DBV, U8 SN74LVC1G126DBV, U9 MCP2518FD-xQBB, Y1 40 MHz

Commit message: fix(PCB): Update MPN and footprint for some passives
Parts:
- R16: MPN RT0805FRE07120RL -> ERJ-PA2J101X; Manufacturer YAGEO -> Panasonic
Changed lines of the file:
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@@
 			)
 		)
-		(property "Datasheet" "https://yageogroup.com/content/datasheet/asset/file/PYU-RT_1-TO-0-01_ROHS_L"
+		(property "Datasheet" "https://industrial.panasonic.com/cdbs/www-data/pdf/RDO0000/AOA0000C331.pdf"
 			(at 43.18 72.39 0)
 			(hide yes)
@@
 			)
 		)
-		(property "Manufacturer" "YAGEO"
+		(property "Manufacturer" "Panasonic"
 			(at 43.18 72.39 0)
 			(hide yes)
@@
 			)
 		)
-		(property "MPN" "RT0805FRE07120RL"
+		(property "MPN" "ERJ-PA2J101X"
 			(at 43.18 72.39 0)
 			(hide yes)
