File: pcb_design/mcu_and_connectors.kicad_sch (KiCad schematic)
At the start: 49 parts, among them J10 Screw_Terminal_01x06, J11 Screw_Terminal_01x06, J12 Screw_Terminal_01x06, J13 Screw_Terminal_01x06, J14 Conn_02x04_Odd_Even, J15 Conn_01x04_MountingPin, J16 Conn_01x06_Socket, J17 Conn_01x06_Socket, J18 Conn_01x03_Pin, J3 Conn_01x02_Socket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

Commit message: fix(PCB): Update MPN and footprint for some passives
Parts:
- C21, C22, C24, C25, C34, C35: footprint Capacitor_SMD:C_0603_1608Metric -> Capacitor_SMD:C_0805_2012Metric
- R18: MPN ERJ-PA2J101X -> ERJ-UP6F1200V
Changed lines of the file:
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@@
 			)
 		)
-		(property "Footprint" "Capacitor_SMD:C_0603_1608Metric"
+		(property "Footprint" "Capacitor_SMD:C_0805_2012Metric"
 			(at 188.9252 33.02 0)
 			(hide yes)
@@
 			)
 		)
-		(property "Footprint" "Capacitor_SMD:C_0603_1608Metric"
+		(property "Footprint" "Capacitor_SMD:C_0805_2012Metric"
 			(at 179.3748 116.84 0)
 			(hide yes)
@@
 			)
 		)
-		(property "Footprint" "Capacitor_SMD:C_0603_1608Metric"
+		(property "Footprint" "Capacitor_SMD:C_0805_2012Metric"
 			(at 180.0352 33.02 0)
 			(hide yes)
@@
 			)
 		)
-		(property "Datasheet" "https://industrial.panasonic.com/cdbs/www-data/pdf/RDO0000/AOA0000C331.pdf"
+		(property "Datasheet" "https://industrial.panasonic.com/cdbs/www-data/pdf/RDP0000/AOA0000C337.pdf"
 			(at 208.28 114.3 0)
 			(hide yes)
@@
 			)
 		)
-		(property "MPN" "ERJ-PA2J101X"
+		(property "MPN" "ERJ-UP6F1200V"
 			(at 208.28 114.3 0)
 			(hide yes)
@@
 			)
 		)
-		(property "Footprint" "Capacitor_SMD:C_0603_1608Metric"
+		(property "Footprint" "Capacitor_SMD:C_0805_2012Metric"
 			(at 131.7752 33.02 0)
 			(hide yes)
@@
 			)
 		)
-		(property "Footprint" "Capacitor_SMD:C_0603_1608Metric"
+		(property "Footprint" "Capacitor_SMD:C_0805_2012Metric"
 			(at 188.2648 116.84 0)
 			(hide yes)
@@
 			)
 		)
-		(property "Footprint" "Capacitor_SMD:C_0603_1608Metric"
+		(property "Footprint" "Capacitor_SMD:C_0805_2012Metric"
 			(at 122.8852 33.02 0)
 			(hide yes)

Commit message: feat(pcb): Add more test points
Parts:
- removed D15, D4: SMF15CA, Diode_SMD:D_SOD-123F, symbol Device:D_TVS
Other:
- moved on the sheet: D16, D5
